File: MixSigCourse-B-KiCad7-Files/MCU.kicad_sch (KiCad schematic)
At the start: 40 parts, among them J200 USB_C_Receptacle_USB2.0, J201 2x5 1.27mm, U200 STM32F103CBT6, U201 USBLC6-2SC6, Y200 16MHz

Commit message: completed the course! board layout complete and gerbers exported
Connections:
- net TIM4_CH1: now also R209.1; no longer R208.1
- net TIM4_CH2: now also R208.1; no longer R209.1
